Commit message: norm vec env

File: models/bittle.urdf (robot description, URDF)
Before this commit: robot bittle, 13 links, 12 joints
Links:
- link base-frame-link: mass 0.108 -> 4

File: models/bittle_modified.urdf (robot description, URDF)
Before this commit: robot bittle, 13 links, 12 joints
Links:
- link base-frame-link: mass 5 -> 0.108
